File: amp/amp.sch (KiCad schematic (older format))
At the start: 68 parts, among them J1 RCA, J3 RCA, SW2 SW_SPDT, SW3 SW_SPDT, T2 Hammond 1608A, T3 Hammond 1608A, U1 6SL7, U2 GZ34, U3 6V6, U4 6V6, U5 6SL7, U6 6V6, U7 6V6

Commit message: assigning part numbers
Parts:
- removed TP1, TP2, TP3, TP4: POST, symbol Connector:TestPoint
- added LS1, LS2: Speaker, BindingPost:Keystone_4109, symbol Device:Speaker
- C1, C9: CatNo (none) -> 399-5448-1-ND
- C10, C2: CatNo (none) -> 732-8598-1-ND
- C11, C3: CatNo (none) -> 493-12650-1-ND
- C12, C13, C4, C5: CatNo (none) -> 338-3444-ND
- C14, C7: CatNo (none) -> 493-12789-1-ND
- C15, C6, C8: CatNo (none) -> 399-15673-ND
- F1: footprint (none) -> HBH_fuse_holder:HBH-I-R; CatNo (none) -> Mouser 504-BK/HBH-I-R
- J1, J3: CatNo (none) -> PJRAN1X1U03X-ND
- J2: renamed from J?; CatNo (none) -> 486-1007-ND
- JP1: renamed from JP?; footprint (none) -> Connector_PinHeader_2.54mm:PinHeader_1x03_P2.54mm_Vertical
- NE1: footprint (none) -> neon:A1A; CatNo (none) -> A1A-ND
- R1, R15: CatNo (none) -> 470KW-1-ND
- R10, R14, R19, R24, R27, R5: CatNo (none) -> RSA-1.0KRCT-ND
- R11, R13, R26: CatNo (none) -> B20J100E-ND
- R12, R25: CatNo (none) -> PPC1D250CT-ND
- R16, R18, R2, R4: CatNo (none) -> 100KW-1-ND
- R17, R3: CatNo (none) -> 100W-1-ND
- R20, R6: CatNo (none) -> 6.8KW-1-ND
- R21, R23, R7, R9: CatNo (none) -> 270KW-1-ND
- R22, R8: CatNo (none) -> 47KW-1-ND
- SW1: renamed from SW?; footprint (none) -> Switch_8GA:8GA1016-Z; CatNo (none) -> 563-1727-ND
- SW2, SW3: CatNo (none) -> 563-1727-ND
- T1: renamed from T?; footprint (none) -> Hammond_XFRMR:Hammond_272HX
- T2, T3: footprint (none) -> Hammond_XFRMR:Hammond_1608A
- U1, U5: footprint Valve:Valve_Noval_P -> tube_sockets:Octal_Socket_P-ST8-193
- U2: footprint (none) -> tube_sockets:Octal_Socket_P-ST8-193
- U3, U4, U6, U7: footprint Valve:Valve_Octal -> tube_sockets:Octal_Socket_P-ST8-193
- gave numbers to parts that had none: 3
Connections:
- net Earth: now also LS1.2, LS2.2
- net at J4.2 (Pin_2), J4.4 (Pin_4), J4.6 (Pin_6): now also LS1.1
- net at J5.2 (Pin_2), J5.4 (Pin_4), J5.6 (Pin_6): now also LS2.1

Commit message: All CatNo filled in
Parts:
- J4, J5: CatNo (none) -> 2057-PH2-06-UA-ND
- JP1: CatNo (none) -> 10129378-903001BLF-ND
- R28: value RRRRR -> 100k; CatNo (none) -> 100KW-1-ND
- T1: CatNo (none) -> HM5012-ND
- T2, T3: CatNo (none) -> HM4113-ND
- U1, U2, U3, U4, U5, U6, U7: CatNo (none) -> AES P-ST8-193
Changed lines of the file:
@@
 F 2 "tube_sockets:Octal_Socket_P-ST8-193" H 4800 2750 50  0001 C CNN
 F 3 "http://www.r-type.org/pdfs/el34.pdf" H 4500 3100 50  0001 C CNN
+F 4 "AES P-ST8-193" H 4500 3100 50  0001 C CNN "CatNo"
 	1    4500 3100
 	1    0    0    -1
@@
 F 2 "tube_sockets:Octal_Socket_P-ST8-193" H 1970 3650 50  0001 C CNN
 F 3 "http://www.r-type.org/pdfs/ecc81.pdf" H 1700 4050 50  0001 C CNN
+F 4 "AES P-ST8-193" H 1700 4050 50  0001 C CNN "CatNo"
 	1    1700 4050
 	1    0    0    -1
@@
 F 2 "tube_sockets:Octal_Socket_P-ST8-193" H 2720 3650 50  0001 C CNN
 F 3 "http://www.r-type.org/pdfs/ecc81.pdf" H 2450 4050 50  0001 C CNN
+F 4 "AES P-ST8-193" H 2450 4050 50  0001 C CNN "CatNo"
 	2    2450 4050
 	-1   0    0    -1
@@
 F 2 "tube_sockets:Octal_Socket_P-ST8-193" H 5800 2750 50  0001 C CNN
 F 3 "http://www.r-type.org/pdfs/el34.pdf" H 5500 3100 50  0001 C CNN
+F 4 "AES P-ST8-193" H 5500 3100 50  0001 C CNN "CatNo"
 	1    5500 3100
 	-1   0    0    -1
@@
 F 2 "Hammond_XFRMR:Hammond_1608A" H 5000 1500 50  0001 C CNN
 F 3 "~" H 5000 1500 50  0001 C CNN
+F 4 "HM4113-ND" H 5000 1500 50  0001 C CNN "CatNo"
 	1    5000 1500
 	0    -1   -1   0
@@
 F 2 "tube_sockets:Octal_Socket_P-ST8-193" H 3350 6750 50  0001 C CNN
 F 3 "" H 3350 6750 50  0001 C CNN
+F 4 "AES P-ST8-193" H 3250 6750 50  0001 C CNN "CatNo"
 	1    3250 6750
 	1    0    0    -1
@@
 F 2 "tube_sockets:Octal_Socket_P-ST8-193" H 6120 6650 50  0001 C CNN
 F 3 "http://www.r-type.org/pdfs/ecc81.pdf" H 5850 7050 50  0001 C CNN
+F 4 "AES P-ST8-193" H 5850 7050 50  0001 C CNN "CatNo"
 	3    5850 7050
 	1    0    0    -1
@@
 F 2 "tube_sockets:Octal_Socket_P-ST8-193" H 10850 2750 50  0001 C CNN
 F 3 "http://www.r-type.org/pdfs/el34.pdf" H 10550 3100 50  0001 C CNN
+F 4 "AES P-ST8-193" H 10550 3100 50  0001 C CNN "CatNo"
 	1    10550 3100
 	1    0    0    -1
@@
 F 2 "tube_sockets:Octal_Socket_P-ST8-193" H 8020 3650 50  0001 C CNN
 F 3 "http://www.r-type.org/pdfs/ecc81.pdf" H 7750 4050 50  0001 C CNN
+F 4 "AES P-ST8-193" H 7750 4050 50  0001 C CNN "CatNo"
 	1    7750 4050
 	1    0    0    -1
@@
 F 2 "tube_sockets:Octal_Socket_P-ST8-193" H 8770 3650 50  0001 C CNN
 F 3 "http://www.r-type.org/pdfs/ecc81.pdf" H 8500 4050 50  0001 C CNN
+F 4 "AES P-ST8-193" H 8500 4050 50  0001 C CNN "CatNo"
 	2    8500 4050
 	-1   0    0    -1
@@
 F 2 "tube_sockets:Octal_Socket_P-ST8-193" H 11850 2750 50  0001 C CNN
 F 3 "http://www.r-type.org/pdfs/el34.pdf" H 11550 3100 50  0001 C CNN
+F 4 "AES P-ST8-193" H 11550 3100 50  0001 C CNN "CatNo"
 	1    11550 3100
 	-1   0    0    -1
@@
 F 2 "Hammond_XFRMR:Hammond_1608A" H 11050 1500 50  0001 C CNN
 F 3 "~" H 11050 1500 50  0001 C CNN
+F 4 "HM4113-ND" H 11050 1500 50  0001 C CNN "CatNo"
 	1    11050 1500
 	0    -1   -1   0
@@
 F 2 "tube_sockets:Octal_Socket_P-ST8-193" H 6920 6650 50  0001 C CNN
 F 3 "http://www.r-type.org/pdfs/ecc81.pdf" H 6650 7050 50  0001 C CNN
+F 4 "AES P-ST8-193" H 6650 7050 50  0001 C CNN "CatNo"
 	3    6650 7050
 	1    0    0    -1
@@
 F 2 "tube_sockets:Octal_Socket_P-ST8-193" H 6150 5550 50  0001 C CNN
 F 3 "http://www.r-type.org/pdfs/el34.pdf" H 5850 5900 50  0001 C CNN
+F 4 "AES P-ST8-193" H 5850 5900 50  0001 C CNN "CatNo"
 	2    5850 5900
 	1    0    0    -1
@@
 F 2 "tube_sockets:Octal_Socket_P-ST8-193" H 6950 5550 50  0001 C CNN
 F 3 "http://www.r-type.org/pdfs/el34.pdf" H 6650 5900 50  0001 C CNN
+F 4 "AES P-ST8-193" H 6650 5900 50  0001 C CNN "CatNo"
 	2    6650 5900
 	1    0    0    -1
@@
 F 2 "tube_sockets:Octal_Socket_P-ST8-193" H 7650 5550 50  0001 C CNN
 F 3 "http://www.r-type.org/pdfs/el34.pdf" H 7350 5900 50  0001 C CNN
+F 4 "AES P-ST8-193" H 7350 5900 50  0001 C CNN "CatNo"
 	2    7350 5900
 	1    0    0    -1
@@
 F 2 "tube_sockets:Octal_Socket_P-ST8-193" H 8450 5550 50  0001 C CNN
 F 3 "http://www.r-type.org/pdfs/el34.pdf" H 8150 5900 50  0001 C CNN
+F 4 "AES P-ST8-193" H 8150 5900 50  0001 C CNN "CatNo"
 	2    8150 5900
 	1    0    0    -1
@@
 F 2 "Hammond_XFRMR:Hammond_272HX" H 2650 6700 50  0001 C CNN
 F 3 "~" H 2650 6700 50  0001 C CNN
+F 4 "HM5012-ND" H 2650 6900 50  0001 C CNN "CatNo"
 	1    2650 6900
 	1    0    0    -1
@@
 F 2 "Connector_PinHeader_2.54mm:PinHeader_1x03_P2.54mm_Vertical" H 2000 6550 50  0001 C CNN
 F 3 "~" H 2000 6550 50  0001 C CNN
+F 4 "10129378-903001BLF-ND" H 2000 6550 50  0001 C CNN "CatNo"
 	1    2000 6550
 	-1   0    0    1
@@
 P 1400 6450
 F 0 "R28" V 1300 6300 50  0000 C CNN
-F 1 "RRRRR" V 1300 6650 50  0000 C CNN
+F 1 "100k" V 1300 6650 50  0000 C CNN
 F 2 "" V 1440 6440 50  0001 C CNN
 F 3 "~" H 1400 6450 50  0001 C CNN
+F 4 "100KW-1-ND" H 1400 6450 50  0001 C CNN "CatNo"
 	1    1400 6450
 	-1   0    0    1
@@
 F 2 "" H 5450 800 50  0001 C CNN
 F 3 "~" H 5450 800 50  0001 C CNN
+F 4 "2057-PH2-06-UA-ND" H 6200 1050 50  0000 C CNN "CatNo"
 	1    5450 800
 	1    0    0    -1
@@
 F 2 "" H 11500 800 50  0001 C CNN
 F 3 "~" H 11500 800 50  0001 C CNN
+F 4 "2057-PH2-06-UA-ND" H 11500 800 50  0001 C CNN "CatNo"
 	1    11500 800
 	1    0    0    -1
@@
 F 2 "BindingPost:Keystone_4109" H 6300 650 50  0001 C CNN
 F 3 "~" H 6290 800 50  0001 C CNN
-F 4 "36-4109-ND" H 6470 709 50  0000 L CNN "CatNo"
+F 4 "36-4109-ND" H 6150 500 50  0000 L CNN "CatNo"
 	1    6300 850
 	1    0    0    -1

Commit message: all footprinted with a few issues
Parts:
- C1, C9: footprint (none) -> Capacitor_THT:C_Rect_L7.2mm_W2.5mm_P5.00mm_FKS2_FKP2_MKS2_MKP2
- C10, C2: footprint (none) -> Capacitor_THT:CP_Radial_D5.0mm_P2.00mm
- C11, C3: footprint (none) -> Capacitor_THT:C_Radial_D12.5mm_H25.0mm_P5.00mm
- C12, C13, C4, C5: footprint (none) -> caps:cap_rect_32x14_P18.3mm
- C14, C7: footprint (none) -> Capacitor_THT:CP_Radial_D12.5mm_P5.00mm
- C15, C6: footprint (none) -> Capacitor_THT:C_Radial_D16.0mm_H25.0mm_P7.50mm
- C8: footprint (none) -> Capacitor_THT:CP_Radial_D16.0mm_P7.50mm
- J1, J3: footprint (none) -> RCA_jack:PJRAS2X1S01AUX
- J4, J5: footprint (none) -> Connector_PinHeader_2.54mm:PinHeader_2x03_P2.54mm_Vertical
- R1, R10, R14, R15, R19, R22, R24, R27, R5, R8: footprint (none) -> Resistor_THT:R_Axial_DIN0411_L9.9mm_D3.6mm_P12.70mm_Horizontal
- R11, R13, R26: footprint (none) -> res:R_100R_20W_11x51mm
- R12, R16, R17, R18, R2, R20, R21, R23, R25, R28, R3, R4, R6, R7, R9: footprint (none) -> Resistor_THT:R_Axial_DIN0414_L11.9mm_D4.5mm_P15.24mm_Horizontal
- SW2, SW3: footprint (none) -> Switch_8GA:8GA1016-Z
