File: amp/amp.sch (KiCad schematic (older format))
At the start: 66 parts, among them J1 RCA, J2 Conn_01x05, J3 RCA, J4 JPR_2x3, J5 JPR_2x3, SW1 SW_SPST_GND, SW2 SW_SPDT, SW3 SW_SPDT, T1 Transformer_Hammond_272HX, T2 Hammond 1608A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

Commit message: placement
Parts:
- C10, C14, C2, C7, C8: symbol Device:C -> Device:CP
- C11, C3: footprint Capacitor_THT:C_Radial_D12.5mm_H25.0mm_P5.00mm -> Capacitor_THT:CP_Radial_D12.5mm_P5.00mm; symbol Device:C -> Device:CP
- C15: footprint Capacitor_THT:C_Radial_D16.0mm_H25.0mm_P7.50mm -> Capacitor_THT:CP_Radial_D16.0mm_P7.50mm; symbol Device:C -> Device:CP
- C6: footprint Capacitor_THT:C_Radial_D16.0mm_H25.0mm_P7.50mm -> Capacitor_THT:CP_Radial_D16.0mm_P7.50mm
- J1, J3: footprint RCA_jack:PJRAS2X1S01AUX -> RCA_jack:PRJAN1X1
- JP1: footprint Connector_PinHeader_2.54mm:PinHeader_1x03_P2.54mm_Vertical -> Connector_Molex:Molex_KK-396_A-41791-0003_1x03_P3.96mm_Vertical; CatNo 10129378-903001BLF-ND -> WM4621-ND
Connections:
- net Earth: now also C10.2, C11.2, C14.2, C15.2, C2.2, C3.2, C7.2, C8.2; no longer C10.1, C11.1, C14.1, C15.1, C2.1, C3.1, C7.1, C8.1
- net at R12.1, U3.8 (F1), U4.8 (F1): now also C7.1; no longer C7.2
- net at R3.1, U1.6 (K): now also C2.1; no longer C2.2
- net at R2.1, R4.1, R6.2: now also C3.1; no longer C3.2
- net at R13.2, R6.1, T2.3 (RED): now also C8.1; no longer C8.2
- net at R25.1, U6.8 (F1), U7.8 (F1): now also C14.1; no longer C14.2
- net at R17.1, U5.6 (K): now also C10.1; no longer C10.2
- net at R16.1, R18.1, R20.2: now also C11.1; no longer C11.2
- net at R20.1, R26.2, T3.3 (RED): now also C15.1; no longer C15.2
Changed lines of the file:
@@
 $EndComp
 $Comp
-L Device:C C7
+L Device:CP C7
 U 1 1 627E7AB4
 P 5150 4050
-F 0 "C7" H 5035 4004 50  0000 R CNN
-F 1 "470u 50V" H 5035 4095 50  0000 R CNN
+F 0 "C7" H 5450 4150 50  0000 R CNN
+F 1 "470u 50V" H 5700 4050 50  0000 R CNN
 F 2 "Capacitor_THT:CP_Radial_D12.5mm_P5.00mm" H 5188 3900 50  0001 C CNN
 F 3 "~" H 5150 4050 50  0001 C CNN
-F 4 "493-12789-1-ND" H 4650 4200 50  0000 C CNN "CatNo"
+F 4 "493-12789-1-ND" H 5650 3950 50  0000 C CNN "CatNo"
 	1    5150 4050
-	-1   0    0    1
+	1    0    0    -1
 $EndComp
 Wire Wire Line
@@
 	2550 4650 2550 4450
 $Comp
-L Device:C C2
+L Device:CP C2
 U 1 1 627EBA42
 P 2550 4850
-F 0 "C2" H 2435 4804 50  0000 R CNN
-F 1 "100u 16V" H 2435 4895 50  0000 R CNN
+F 0 "C2" H 2800 5000 50  0000 R CNN
+F 1 "100u 16V" H 3050 4900 50  0000 R CNN
 F 2 "Capacitor_THT:CP_Radial_D5.0mm_P2.00mm" H 2588 4700 50  0001 C CNN
 F 3 "~" H 2550 4850 50  0001 C CNN
-F 4 "732-8598-1-ND" H 2100 5000 50  0000 C CNN "CatNo"
+F 4 "732-8598-1-ND" H 3000 4800 50  0000 C CNN "CatNo"
 	1    2550 4850
-	-1   0    0    1
+	1    0    0    -1
 $EndComp
 Wire Wire Line
@@
 	5400 1050 5400 1100
 $Comp
-L Device:C C3
+L Device:CP C3
 U 1 1 6281671B
 P 2750 2400
-F 0 "C3" H 2635 2354 50  0000 R CNN
-F 1 "22u 350V" H 2635 2445 50  0000 R CNN
-F 2 "Capacitor_THT:C_Radial_D12.5mm_H25.0mm_P5.00mm" H 2788 2250 50  0001 C CNN
+F 0 "C3" H 3000 2450 50  0000 R CNN
+F 1 "22u 350V" H 3250 2300 50  0000 R CNN
+F 2 "Capacitor_THT:CP_Radial_D12.5mm_P5.00mm" H 2788 2250 50  0001 C CNN
 F 3 "~" H 2750 2400 50  0001 C CNN
-F 4 "493-12650-1-ND" H 2300 2550 50  0000 C CNN "CatNo"
+F 4 "493-12650-1-ND" H 3200 2200 50  0000 C CNN "CatNo"
 	1    2750 2400
-	-1   0    0    1
+	1    0    0    -1
 $EndComp
 $Comp
@@
 B+
 $Comp
-L Device:C C8
+L Device:CP C8
 U 1 1 628301D6
 P 5850 2400
-F 0 "C8" H 5735 2354 50  0000 R CNN
-F 1 "47u 450V" H 5735 2445 50  0000 R CNN
+F 0 "C8" H 6150 2450 50  0000 R CNN
+F 1 "47u 450V" H 6400 2350 50  0000 R CNN
 F 2 "Capacitor_THT:CP_Radial_D16.0mm_P7.50mm" H 5888 2250 50  0001 C CNN
 F 3 "~" H 5850 2400 50  0001 C CNN
-F 4 "399-15673-ND" H 5450 2550 50  0000 C CNN "CatNo"
+F 4 "399-15673-ND" H 6350 2250 50  0000 C CNN "CatNo"
 	1    5850 2400
-	-1   0    0    1
+	1    0    0    -1
 $EndComp
 $Comp
@@
 F 0 "J1" H 628 4288 50  0000 C CNN
 F 1 "RCA" H 628 4197 50  0000 C CNN
-F 2 "RCA_jack:PJRAS2X1S01AUX" H 700 4050 50  0001 C CNN
+F 2 "RCA_jack:PRJAN1X1" H 700 4050 50  0001 C CNN
 F 3 " ~" H 700 4050 50  0001 C CNN
 F 4 "PJRAN1X1U03X-ND" H 700 4050 50  0001 C CNN "CatNo"
@@
 F 0 "C6" H 5042 7096 50  0000 L CNN
 F 1 "47uF 450V" H 5042 7005 50  0000 L CNN
-F 2 "Capacitor_THT:C_Radial_D16.0mm_H25.0mm_P7.50mm" H 4950 7050 50  0001 C CNN
+F 2 "Capacitor_THT:CP_Radial_D16.0mm_P7.50mm" H 4950 7050 50  0001 C CNN
 F 3 "~" H 4950 7050 50  0001 C CNN
 F 4 "399-15673-ND" H 5300 6900 50  0000 C CNN "CatNo"
@@
 U 1 1 62A5A5FB
 P 10800 4050
-F 0 "R25" H 10868 4096 50  0000 L CNN
-F 1 "250" H 10868 4005 50  0000 L CNN
+F 0 "R25" H 10550 4100 50  0000 L CNN
+F 1 "250" H 10550 3950 50  0000 L CNN
 F 2 "Resistor_THT:R_Axial_DIN0414_L11.9mm_D4.5mm_P15.24mm_Horizontal" V 10840 4040 50  0001 C CNN
 F 3 "~" H 10800 4050 50  0001 C CNN
@@
 $EndComp
 $Comp
-L Device:C C14
+L Device:CP C14
 U 1 1 62A5A605
 P 11200 4050
-F 0 "C14" H 11085 4004 50  0000 R CNN
-F 1 "470u 50V" H 11085 4095 50  0000 R CNN
+F 0 "C14" H 11550 4050 50  0000 R CNN
+F 1 "470u 50V" H 11750 3950 50  0000 R CNN
 F 2 "Capacitor_THT:CP_Radial_D12.5mm_P5.00mm" H 11238 3900 50  0001 C CNN
 F 3 "~" H 11200 4050 50  0001 C CNN
 F 4 "493-12789-1-ND" H 11200 4050 50  0001 C CNN "CatNo"
 	1    11200 4050
-	-1   0    0    1
+	1    0    0    -1
 $EndComp
 Wire Wire Line
@@
 	8600 4650 8600 4450
 $Comp
-L Device:C C10
+L Device:CP C10
 U 1 1 62A5A633
 P 8600 4900
@@
 F 4 "732-8598-1-ND" H 8600 4900 50  0001 C CNN "CatNo"
 	1    8600 4900
-	-1   0    0    1
+	1    0    0    -1
 $EndComp
 Wire Wire Line
@@
 	11450 1050 11450 1100
 $Comp
-L Device:C C11
+L Device:CP C11
 U 1 1 62A5A69F
 P 8800 2400
-F 0 "C11" H 8685 2354 50  0000 R CNN
-F 1 "22u 350V" H 8685 2445 50  0000 R CNN
-F 2 "Capacitor_THT:C_Radial_D12.5mm_H25.0mm_P5.00mm" H 8838 2250 50  0001 C CNN
+F 0 "C11" H 9100 2450 50  0000 R CNN
+F 1 "22u 350V" H 9350 2350 50  0000 R CNN
+F 2 "Capacitor_THT:CP_Radial_D12.5mm_P5.00mm" H 8838 2250 50  0001 C CNN
 F 3 "~" H 8800 2400 50  0001 C CNN
 F 4 "493-12650-1-ND" H 8800 2400 50  0001 C CNN "CatNo"
 	1    8800 2400
-	-1   0    0    1
+	1    0    0    -1
 $EndComp
 $Comp
@@
 B+
 $Comp
-L Device:C C15
+L Device:CP C15
 U 1 1 62A5A6C6
 P 11900 2400
-F 0 "C15" H 11785 2354 50  0000 R CNN
-F 1 "47u 450V" H 11785 2445 50  0000 R CNN
-F 2 "Capacitor_THT:C_Radial_D16.0mm_H25.0mm_P7.50mm" H 11938 2250 50  0001 C CNN
+F 0 "C15" H 12200 2400 50  0000 R CNN
+F 1 "47u 450V" H 12400 2300 50  0000 R CNN
+F 2 "Capacitor_THT:CP_Radial_D16.0mm_P7.50mm" H 11938 2250 50  0001 C CNN
 F 3 "~" H 11900 2400 50  0001 C CNN
 F 4 "399-15673-ND" H 11900 2400 50  0001 C CNN "CatNo"
 	1    11900 2400
-	-1   0    0    1
+	1    0    0    -1
 $EndComp
 $Comp
@@
 F 0 "J3" H 6678 4288 50  0000 C CNN
 F 1 "RCA" H 6678 4197 50  0000 C CNN
-F 2 "RCA_jack:PJRAS2X1S01AUX" H 6750 4050 50  0001 C CNN
+F 2 "RCA_jack:PRJAN1X1" H 6750 4050 50  0001 C CNN
 F 3 " ~" H 6750 4050 50  0001 C CNN
 F 4 "PJRAN1X1U03X-ND" H 6750 4050 50  0001 C CNN "CatNo"
@@
 F 0 "JP1" H 2000 6697 50  0000 C CNN
 F 1 "JPR3" H 2000 6788 50  0000 C CNN
-F 2 "Connector_PinHeader_2.54mm:PinHeader_1x03_P2.54mm_Vertical" H 2000 6550 50  0001 C CNN
+F 2 "Connector_Molex:Molex_KK-396_A-41791-0003_1x03_P3.96mm_Vertical" H 2000 6550 50  0001 C CNN
 F 3 "~" H 2000 6550 50  0001 C CNN
-F 4 "10129378-903001BLF-ND" H 2000 6550 50  0001 C CNN "CatNo"
+F 4 "WM4621-ND" H 2000 6550 50  0001 C CNN "CatNo"
 	1    2000 6550
 	-1   0    0    1

Commit message: starting 3D
Parts:
- added H1, H2, H3, H4: MountingHole, MountingHolesInch:Mtg6-32, symbol Mechanical:MountingHole
Changed lines of the file:
@@
 Wire Wire Line
 	11750 1050 12100 1050
+$Comp
+L Mechanical:MountingHole H1
+U 1 1 62D80DE1
+P 9550 5750
+F 0 "H1" H 9650 5796 50  0000 L CNN
+F 1 "MountingHole" H 9650 5705 50  0000 L CNN
+F 2 "MountingHolesInch:Mtg6-32" H 9550 5750 50  0001 C CNN
+F 3 "~" H 9550 5750 50  0001 C CNN
+	1    9550 5750
+	1    0    0    -1
+$EndComp
+$Comp
+L Mechanical:MountingHole H2
+U 1 1 62D8CF59
+P 9550 6000
+F 0 "H2" H 9650 6046 50  0000 L CNN
+F 1 "MountingHole" H 9650 5955 50  0000 L CNN
+F 2 "MountingHolesInch:Mtg6-32" H 9550 6000 50  0001 C CNN
+F 3 "~" H 9550 6000 50  0001 C CNN
+	1    9550 6000
+	1    0    0    -1
+$EndComp
+$Comp
+L Mechanical:MountingHole H3
+U 1 1 62D8D904
+P 9550 6250
+F 0 "H3" H 9650 6296 50  0000 L CNN
+F 1 "MountingHole" H 9650 6205 50  0000 L CNN
+F 2 "MountingHolesInch:Mtg6-32" H 9550 6250 50  0001 C CNN
+F 3 "~" H 9550 6250 50  0001 C CNN
+	1    9550 6250
+	1    0    0    -1
+$EndComp
+$Comp
+L Mechanical:MountingHole H4
+U 1 1 62D8E11D
+P 9550 6500
+F 0 "H4" H 9650 6546 50  0000 L CNN
+F 1 "MountingHole" H 9650 6455 50  0000 L CNN
+F 2 "MountingHolesInch:Mtg6-32" H 9550 6500 50  0001 C CNN
+F 3 "~" H 9550 6500 50  0001 C CNN
+	1    9550 6500
+	1    0    0    -1
+$EndComp
 $EndSCHEMATC

Commit message: tweaks
Connections:
- net B+PRE_L: now reaches C3.1, R2.1, R4.1, R6.2
- net B+PP_L: now reaches C8.1, R13.2, R6.1, T2.3 (RED)
- net B+PRE_R: now reaches C11.1, R16.1, R18.1, R20.2
- net B+PP_R: now reaches C15.1, R20.1, R26.2, T3.3 (RED)
Changed lines of the file:
@@
 	1    0    0    -1
 $EndComp
+Text Label 1950 2200 0    50   ~ 0
+B+PRE_L
+Text Label 7950 2200 0    50   ~ 0
+B+PRE_R
+Text Label 3650 2200 0    50   ~ 0
+B+PP_L
+Text Label 9700 2200 0    50   ~ 0
+B+PP_R
 $EndSCHEMATC
