File: amp/amp.kicad_pcb (KiCad board)
At the start: 2 copper layers, 66 parts, among them J1 RCA, J2 Conn_01x05, J3 RCA, J4 JPR_2x3, J5 JPR_2x3, SW1 SW_SPST_GND, SW2 SW_SPDT, SW3 SW_SPDT, T1 Transformer_Hammond_272HX, T2 Hammond 1608A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

Commit message: placement
Parts:
- C11, C3: footprint Capacitor_THT:C_Radial_D12.5mm_H25.0mm_P5.00mm -> Capacitor_THT:CP_Radial_D12.5mm_P5.00mm
- C15, C6: footprint Capacitor_THT:C_Radial_D16.0mm_H25.0mm_P7.50mm -> Capacitor_THT:CP_Radial_D16.0mm_P7.50mm
- J1, J3: footprint RCA_jack:PJRAS2X1S01AUX -> RCA_jack:PRJAN1X1
- JP1: footprint Connector_PinHeader_2.54mm:PinHeader_1x03_P2.54mm_Vertical -> Connector_Molex:Molex_KK-396_A-41791-0003_1x03_P3.96mm_Vertical
- moved J3 651.1 mm to (641.4, 35.8), turned to 180 degrees
- moved LS2 490.6 mm to (340.4, 15.2), turned to 180 degrees
- moved R15 474.8 mm to (631.2, 16.5)
- moved LS1 440.8 mm to (200.7, 15.2), turned to 180 degrees
- moved J5 437.5 mm to (332.7, 45.7), turned to 270 degrees
- moved C10 422.9 mm to (591.5, 310.6)
- moved C11 422.9 mm to (611.2, 325.0)
- moved C9 422.9 mm to (527.8, 290.4)
- moved R17 422.9 mm to (526.2, 329.9)
- moved R18 422.9 mm to (545.4, 329.9)
- moved R20 422.9 mm to (534.1, 270.5)
- moved R21 422.9 mm to (468.6, 329.3)
- moved R23 422.9 mm to (507.0, 329.9)
- moved R25 422.9 mm to (600.3, 278.5)
- moved R26 422.9 mm to (429.5, 288.9)
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Connections:
- C10 pad 1: Earth -> Net-(C10-Pad1)
- C10 pad 2: Net-(C10-Pad2) -> Earth
- C11 pad 1: Earth -> Net-(C11-Pad1)
- C11 pad 2: Net-(C11-Pad2) -> Earth
- C14 pad 1: Earth -> Net-(C14-Pad1)
- C14 pad 2: Net-(C14-Pad2) -> Earth
- C15 pad 1: Earth -> Net-(C15-Pad1)
- C15 pad 2: Net-(C15-Pad2) -> Earth
- C2 pad 1: Earth -> Net-(C2-Pad1)
- C2 pad 2: Net-(C2-Pad2) -> Earth
- C3 pad 1: Earth -> Net-(C3-Pad1)
- C3 pad 2: Net-(C3-Pad2) -> Earth
- C7 pad 1: Earth -> Net-(C7-Pad1)
- C7 pad 2: Net-(C7-Pad2) -> Earth
- C8 pad 1: Earth -> Net-(C8-Pad1)
- C8 pad 2: Net-(C8-Pad2) -> Earth
- R12 pad 1: Net-(C7-Pad2) -> Net-(C7-Pad1)
- R13 pad 2: Net-(C8-Pad2) -> Net-(C8-Pad1)
- R16 pad 1: Net-(C11-Pad2) -> Net-(C11-Pad1)
- R17 pad 1: Net-(C10-Pad2) -> Net-(C10-Pad1)
- R18 pad 1: Net-(C11-Pad2) -> Net-(C11-Pad1)
- R2 pad 1: Net-(C3-Pad2) -> Net-(C3-Pad1)
- R20 pad 1: Net-(C15-Pad2) -> Net-(C15-Pad1)
- R20 pad 2: Net-(C11-Pad2) -> Net-(C11-Pad1)
- R25 pad 1: Net-(C14-Pad2) -> Net-(C14-Pad1)
- R26 pad 2: Net-(C15-Pad2) -> Net-(C15-Pad1)
- R3 pad 1: Net-(C2-Pad2) -> Net-(C2-Pad1)
- R4 pad 1: Net-(C3-Pad2) -> Net-(C3-Pad1)
- R6 pad 1: Net-(C8-Pad2) -> Net-(C8-Pad1)
- R6 pad 2: Net-(C3-Pad2) -> Net-(C3-Pad1)
- T2 pad 3: Net-(C8-Pad2) -> Net-(C8-Pad1)
- T3 pad 3: Net-(C15-Pad2) -> Net-(C15-Pad1)
- U1 pad 6: Net-(C2-Pad2) -> Net-(C2-Pad1)
- U3 pad 8: Net-(C7-Pad2) -> Net-(C7-Pad1)
- U4 pad 8: Net-(C7-Pad2) -> Net-(C7-Pad1)
- U5 pad 6: Net-(C10-Pad2) -> Net-(C10-Pad1)
- U6 pad 8: Net-(C14-Pad2) -> Net-(C14-Pad1)
- U7 pad 8: Net-(C14-Pad2) -> Net-(C14-Pad1)
Other:
- board outline added: 406.4 x 330.2 mm

Commit message: starting 3D
Parts:
- added H1: MountingHole, MountingHolesInch:Mtg6-32, F.Cu at (5.08, 274.3)
- added H2: MountingHole, MountingHolesInch:Mtg6-32, F.Cu at (401.3, 274.3)
- added H3: MountingHole, MountingHolesInch:Mtg6-32, F.Cu at (5.08, 5.08)
- added H4: MountingHole, MountingHolesInch:Mtg6-32, F.Cu at (401.3, 5.08)
- moved R28 515.5 mm to (53.8, 260.1)
- moved SW3 367.7 mm to (363.2, 17.8), turned to 270 degrees
- moved U5 292.1 mm to (330.2, 237.2), turned to 180 degrees
- moved R26 282.2 mm to (266.7, 58.4), turned to 270 degrees
- moved C11 271.3 mm to (457.2, 101.6)
- moved C15 262.7 mm to (266.7, 146.1), turned to 90 degrees
- moved C10 261.5 mm to (421.6, 111.8)
- moved C13 239.2 mm to (426.5, 260.9)
- moved C12 239.2 mm to (426.5, 245.7)
- moved R18 233.4 mm to (421.6, 132.1)
- moved C9 231.1 mm to (419.1, 86.4)
- moved R27 228.2 mm to (457.2, 147.3)
- moved U6 207.4 mm to (285.8, 186.4), turned to 270 degrees
- moved R25 206.6 mm to (455.5, 131.2)
- moved R17 204.8 mm to (424.2, 152.4)
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Other:
- board size 406.4 x 330.2 mm -> 406.4 x 279.4 mm
