File: amp/amp.kicad_sch (KiCad schematic)
At the start: 70 parts, among them J1 RCA, J2 Conn_01x05, J3 RCA, J4 JPR_2x3, J5 JPR_2x3, SW1 SW_SPST_GND, SW2 SW_SPDT, SW3 SW_SPDT, T1 Transformer_Hammond_272HX, T2 Hammond 1608A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

Commit message: notes and add grid stoppers to schem
Parts:
- added R29, R30: 10k, Resistor_THT:R_Axial_DIN0414_L11.9mm_D4.5mm_P15.24mm_Horizontal, symbol Device:R_US
Connections:
- net at J1.1 (In), R1.1: now also R29.2; no longer U1.1 (G)
- net at J3.1 (In), R15.1: now also R30.2; no longer U5.1 (G)
- new net: R29.1, U1.1 (G)
- new net: R30.1, U5.1 (G)
Other:
- note added: "6V6 Push-Pull Stereo Amplifier"
- note removed: "6SL7 Push-Pull Stereo Amplifier"
Changed lines of the file:
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@@
 		)
 	)
-	(text "6SL7 Push-Pull Stereo Amplifier"
+	(text "6V6 Push-Pull Stereo Amplifier"
 		(exclude_from_sim no)
 		(at 226.06 180.34 0)
@@
 	)
 	(junction
-		(at 22.86 102.87)
-		(diameter 0)
-		(color 0 0 0 0)
-	)
-	(junction
 		(at 223.52 55.88)
 		(diameter 0)
@@
 	)
 	(junction
+		(at 22.86 102.87)
+		(diameter 0)
+		(color 0 0 0 0)
+	)
+	(junction
 		(at 299.72 20.32)
 		(diameter 0)
@@
 	)
 	(junction
+		(at 176.53 102.87)
+		(diameter 0)
+		(color 0 0 0 0)
+	)
+	(junction
 		(at 284.48 93.98)
 		(diameter 0)
@@
 	)
 	(junction
-		(at 176.53 102.87)
-		(diameter 0)
-		(color 0 0 0 0)
-	)
-	(junction
 		(at 146.05 165.1)
 		(diameter 0)
@@
 	(wire
 		(pts
-			(xy 189.23 102.87) (xy 176.53 102.87)
-		)
-		(stroke
-			(width 0)
-			(type default)
-		)
-	)
-	(wire
-		(pts
 			(xy 241.3 102.87) (xy 246.38 102.87)
 		)
@@
 	(wire
 		(pts
-			(xy 35.56 102.87) (xy 22.86 102.87)
-		)
-		(stroke
-			(width 0)
-			(type default)
-		)
-	)
-	(wire
-		(pts
 			(xy 232.41 80.01) (xy 246.38 80.01)
 		)
@@
 	(wire
 		(pts
+			(xy 186.69 102.87) (xy 189.23 102.87)
+		)
+		(stroke
+			(width 0)
+			(type default)
+		)
+	)
+	(wire
+		(pts
 			(xy 189.23 162.56) (xy 189.23 160.02)
 		)
@@
 	(wire
 		(pts
+			(xy 176.53 102.87) (xy 179.07 102.87)
+		)
+		(stroke
+			(width 0)
+			(type default)
+		)
+	)
+	(wire
+		(pts
 			(xy 265.43 93.98) (xy 274.32 93.98)
 		)
@@
 	(wire
 		(pts
+			(xy 22.86 102.87) (xy 25.4 102.87)
+		)
+		(stroke
+			(width 0)
+			(type default)
+		)
+	)
+	(wire
+		(pts
 			(xy 123.19 171.45) (xy 125.73 171.45)
 		)
@@
 	(wire
 		(pts
+			(xy 33.02 102.87) (xy 35.56 102.87)
+		)
+		(stroke
+			(width 0)
+			(type default)
+		)
+	)
+	(wire
+		(pts
 			(xy 22.86 161.29) (xy 30.48 161.29)
 		)
@@
 					(unit 1)
 				)
+			)
+		)
+	)
+	(symbol
+		(lib_id "Device:R_US")
+		(at 29.21 102.87 270)
+		(unit 1)
+		(exclude_from_sim no)
+		(in_bom yes)
+		(on_board yes)
+		(dnp no)
+		(property "Reference" "R29"
+			(at 29.21 97.663 90)
+			(effects
+				(font
+					(size 1.27 1.27)
+				)
+			)
+		)
+		(property "Value" "10k"
+			(at 29.21 99.9744 90)
+			(effects
+				(font
+					(size 1.27 1.27)
+				)
+			)
+		)
+		(property "Footprint" "Resistor_THT:R_Axial_DIN0414_L11.9mm_D4.5mm_P15.24mm_Horizontal"
+			(at 28.956 103.886 90)
+			(effects
+				(font
+					(size 1.27 1.27)
+				)
+				(hide yes)
+			)
+		)
+		(property "Datasheet" "~"
+			(at 29.21 102.87 0)
+			(effects
+				(font
+					(size 1.27 1.27)
+				)
+				(hide yes)
+			)
+		)
+		(property "Description" ""
+			(at 29.21 102.87 0)
+			(effects
+				(font
+					(size 1.27 1.27)
+				)
+			)
+		)
+		(property "CatNo" ""
+			(at 31.75 95.25 90)
+			(effects
+				(font
+					(size 1.27 1.27)
+				)
+			)
+		)
+		(pin "1"
+		)
+		(pin "2"
+		)
+		(instances
+			(project "amp"
+				(path "/1226cee2-82be-487a-baac-f8a71896f140"
+					(reference "R29")
+					(unit 1)
+				)
+			)
+		)
+	)
+	(symbol
+		(lib_id "Device:R_US")
+		(at 182.88 102.87 270)
+		(unit 1)
+		(exclude_from_sim no)
+		(in_bom yes)
+		(on_board yes)
+		(dnp no)
+		(property "Reference" "R30"
+			(at 182.88 97.663 90)
+			(effects
+				(font
+					(size 1.27 1.27)
+				)
+			)
+		)
+		(property "Value" "10k"
+			(at 182.88 99.9744 90)
+			(effects
+				(font
+					(size 1.27 1.27)
+				)
+			)
+		)
+		(property "Footprint" "Resistor_THT:R_Axial_DIN0414_L11.9mm_D4.5mm_P15.24mm_Horizontal"
+			(at 182.626 103.886 90)
+			(effects
+				(font
+					(size 1.27 1.27)
+				)
+				(hide yes)
+			)
+		)
+		(property "Datasheet" "~"
+			(at 182.88 102.87 0)
+			(effects
+				(font
+					(size 1.27 1.27)
+				)
+				(hide yes)
+			)
+		)
+		(property "Description" ""
+			(at 182.88 102.87 0)
+			(effects
+				(font
+					(size 1.27 1.27)
+				)
+			)
+		)
+		(property "CatNo" ""
+			(at 185.42 95.25 90)
+			(effects
+				(font
+					(size 1.27 1.27)
+				)
+			)
+		)
+		(pin "1"
+		)
+		(pin "2"
+		)
+		(instances
+			(project "amp"
+				(path "/1226cee2-82be-487a-baac-f8a71896f140"
+					(reference "R30")
+					(unit 1)
+				)
